File: Hardware/ESP32-C6_Qwiic_Micro.sch (EAGLE design)
At the start: 53 parts, among them J1 USB Female Type C Connector, J4 QWIIC_RIGHT_ANGLE, Q1 20V/4.2A/52mΩ/1.4W, U1 ESP32-C6-MINI-1, U2 RT9080-33GJ5, U3 MCP73831

Commit message: Design review updates
Add voltage regulator voltage and current maximums
Add 4-layer stackup info to ordering instructions
Add info about boot button usage
Fix blue LED resistor value
Nudge N$14 to get GND to connect to battery pad
Add tRestrict between C1 and C2
Fix acid traps
Parts:
- R2: value 4.7k -> 2.2k; device SparkFun-Resistors:4.7KOHM-0402T-1/16W-1% -> SparkFun-Resistors:2.2KOHM-0402T-1/16W-1%
Other:
- note added: "To enter bootloader, hold BOOT button when ESP32 resets or powers on"
- note added: "Voltage Input Max: 5.5V Current Max: 600mA"
Changed lines of the file:
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@@
 <part name="D2" library="SparkFun-LED" deviceset="LED-BLUE" device="0603" value="BLUE"/>
 <part name="R1" library="SparkFun-Resistors" deviceset="4.7KOHM" device="-0402T-1/16W-1%" value="4.7k"/>
-<part name="R2" library="SparkFun-Resistors" deviceset="4.7KOHM" device="-0402T-1/16W-1%" value="4.7k"/>
+<part name="R2" library="SparkFun-Resistors" deviceset="2.2KOHM" device="-0402T-1/16W-1%" value="2.2k"/>
 <part name="PWR" library="SparkFun-Jumpers" deviceset="JUMPER-SMT_2_NC_TRACE" device="_SILK" package3d_urn="urn:adsk.eagle:package:39281/1"/>
 <part name="GND7" library="SparkFun-PowerSymbols" deviceset="GND" device=""/>
@@
 <text x="226.06" y="124.46" size="2.54" layer="94" font="vector" align="center">Test Points</text>
 <wire x1="200.66" y1="129.54" x2="200.66" y2="91.44" width="0.2032" layer="97" style="longdash"/>
+<text x="116.84" y="167.64" size="1.778" layer="97" font="vector" align="center">Voltage Input Max: 5.5V
+Current Max: 600mA</text>
+<text x="124.46" y="106.68" size="1.778" layer="97" font="vector" align="center">To enter bootloader, hold
+BOOT button when ESP32
+resets or powers on</text>
 </plain>
 <instances>
