File: Hardware/Qwiic_Pocket_Dev_ESP32_C6.brd (EAGLE design)
At the start: 25.4 x 25.4 mm, 96 parts, among them J1 USB Female Type C Connector, J4 QWIIC_RIGHT_ANGLE, Q1 20V/4.2A/52mΩ/1.4W, U1 ESP32-C6-MINI-1, U2 RT9080-33GJ5, U3 MCP73831

Commit message: Change battery voltage divider resistors to 1M Ohm
Parts:
- R13, R14: value 100k -> 1M
Changed lines of the file:
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@@
 <element name="U$25" library="output" package="QWIIC_DEV0" value="" x="4.445" y="20.574" smashed="yes"/>
 <element name="U$9" library="output" package="QWIIC_DEV0" value="" x="21.336" y="4.826" smashed="yes" rot="MR0"/>
-<element name="R13" library="SparkFun-Resistors" package="0402-TIGHT" value="100k" x="13.208" y="13.97" smashed="yes" rot="R90">
+<element name="R13" library="SparkFun-Resistors" package="0402-TIGHT" value="1M" x="13.208" y="13.97" smashed="yes" rot="R90">
 <attribute name="NAME" x="12.646" y="13.97" size="0.6096" layer="25" font="vector" ratio="20" rot="R90" align="bottom-center"/>
-<attribute name="PROD_ID" value="RES-13495" x="13.208" y="13.97" size="1.778" layer="27" rot="R90" display="off"/>
-<attribute name="VALUE" x="13.77" y="13.97" size="0.6096" layer="27" font="vector" ratio="20" rot="R90" align="top-center"/>
+<attribute name="PROD_ID" value="RES-15185" x="13.208" y="13.97" size="1.778" layer="27" rot="R90" display="off"/>
+<attribute name="VALUE" value="1M" x="13.77" y="13.97" size="0.6096" layer="27" font="vector" ratio="20" rot="R90" align="top-center"/>
 </element>
-<element name="R14" library="SparkFun-Resistors" package="0402-TIGHT" value="100k" x="12.192" y="13.97" smashed="yes" rot="R270">
+<element name="R14" library="SparkFun-Resistors" package="0402-TIGHT" value="1M" x="12.192" y="13.97" smashed="yes" rot="R270">
 <attribute name="NAME" x="12.754" y="13.97" size="0.6096" layer="25" font="vector" ratio="20" rot="R270" align="bottom-center"/>
-<attribute name="PROD_ID" value="RES-13495" x="12.192" y="13.97" size="1.778" layer="27" rot="R270" display="off"/>
-<attribute name="VALUE" x="11.63" y="13.97" size="0.6096" layer="27" font="vector" ratio="20" rot="R270" align="top-center"/>
+<attribute name="PROD_ID" value="RES-15185" x="12.192" y="13.97" size="1.778" layer="27" rot="R270" display="off"/>
+<attribute name="VALUE" value="1M" x="11.63" y="13.97" size="0.6096" layer="27" font="vector" ratio="20" rot="R270" align="top-center"/>
 </element>
 <element name="U$28" library="output" package="IO230" value="" x="5.08" y="2.159" smashed="yes" rot="R90"/>

Commit message: Change C6 to DNP
Rise time was slow, causing chip to run bootloader instead of booting from flash
Parts:
- C6: value 0.1uF -> DNP
Changed lines of the file:
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@@
 <attribute name="VALUE" x="14.678" y="7.62" size="0.6096" layer="27" font="vector" ratio="20" rot="R270" align="top-center"/>
 </element>
-<element name="C6" library="SparkFun-Capacitors" package="0402-TIGHT" value="0.1uF" x="10.16" y="7.62" smashed="yes" rot="R270">
+<element name="C6" library="SparkFun-Capacitors" package="0402-TIGHT" value="DNP" x="10.16" y="7.62" smashed="yes" rot="R270">
 <attribute name="NAME" x="10.722" y="7.62" size="0.6096" layer="25" font="vector" ratio="20" rot="R270" align="bottom-center"/>
-<attribute name="PROD_ID" value="CAP-14993" x="10.16" y="7.62" size="1.778" layer="27" font="vector" ratio="15" rot="R270" display="off"/>
+<attribute name="PROD_ID" value="" x="10.16" y="7.62" size="1.778" layer="27" font="vector" ratio="15" rot="R270" display="off"/>
 <attribute name="VALUE" x="9.598" y="7.62" size="0.6096" layer="27" font="vector" ratio="20" rot="R270" align="top-center"/>
 </element>
