File: Production/Qwiic_Pocket_Dev_ESP32_C6-Panel.brd (EAGLE design)
At the start: 116.8 x 157.5 mm, 1906 parts, among them J1 USB Female Type C Connector, J10 QWIIC_RIGHT_ANGLE, J100 QWIIC_RIGHT_ANGLE, J11 USB Female Type C Connector, J15 QWIIC_RIGHT_ANGLE, J16 USB Female Type C Connector, J20 QWIIC_RIGHT_ANGLE, J21 USB Female Type C Connector, J25 QWIIC_RIGHT_ANGLE, J26 USB Female Type C Connector, J30 QWIIC_RIGHT_ANGLE, J31 USB Female Type C Connector, J35 QWIIC_RIGHT_ANGLE, J36 USB Female Type C Connector, J4 QWIIC_RIGHT_ANGLE, J40 QWIIC_RIGHT_ANGLE, J41 USB Female Type C Connector, J45 QWIIC_RIGHT_ANGLE, J46 USB Female Type C Connector, J50 QWIIC_RIGHT_ANGLE, J51 USB Female Type C Connector, J55 QWIIC_RIGHT_ANGLE, J56 USB Female Type C Connector, J6 USB Female Type C Connector, J60 QWIIC_RIGHT_ANGLE, J61 USB Female Type C Connector, J65 QWIIC_RIGHT_ANGLE, J66 USB Female Type C Connector, J70 QWIIC_RIGHT_ANGLE, J71 USB Female Type C Connector, J75 QWIIC_RIGHT_ANGLE, J76 USB Female Type C Connector, J80 QWIIC_RIGHT_ANGLE, J81 USB Female Type C Connector, J85 QWIIC_RIGHT_ANGLE, J86 USB Female Type C Connector, J90 QWIIC_RIGHT_ANGLE, J91 USB Female Type C Connector, J95 QWIIC_RIGHT_ANGLE, J96 USB Female Type C Connector, Q1 20V/4.2A/52mΩ/1.4W, Q10 20V/4.2A/52mΩ/1.4W, Q11 20V/4.2A/52mΩ/1.4W, Q12 20V/4.2A/52mΩ/1.4W, Q13 20V/4.2A/52mΩ/1.4W, Q14 20V/4.2A/52mΩ/1.4W, Q15 20V/4.2A/52mΩ/1.4W, Q16 20V/4.2A/52mΩ/1.4W, Q17 20V/4.2A/52mΩ/1.4W, Q18 20V/4.2A/52mΩ/1.4W, Q19 20V/4.2A/52mΩ/1.4W, Q2 20V/4.2A/52mΩ/1.4W, Q20 20V/4.2A/52mΩ/1.4W, Q3 20V/4.2A/52mΩ/1.4W, Q4 20V/4.2A/52mΩ/1.4W, Q5 20V/4.2A/52mΩ/1.4W, Q6 20V/4.2A/52mΩ/1.4W, Q7 20V/4.2A/52mΩ/1.4W, Q8 20V/4.2A/52mΩ/1.4W, Q9 20V/4.2A/52mΩ/1.4W, U1 ESP32-C6-MINI-1, U10 ESP32-C6-MINI-1, U11 RT9080-33GJ5, U12 MCP73831, U13 ESP32-C6-MINI-1, U14 RT9080-33GJ5, U15 MCP73831, U16 ESP32-C6-MINI-1, U17 RT9080-33GJ5, U18 MCP73831, U19 ESP32-C6-MINI-1, U2 RT9080-33GJ5, U20 RT9080-33GJ5, U21 MCP73831, U22 ESP32-C6-MINI-1, U23 RT9080-33GJ5, U24 MCP73831, U25 ESP32-C6-MINI-1, U26 RT9080-33GJ5, U27 MCP73831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

Commit message: Change battery voltage divider resistors to 1M Ohm
Parts:
- R111, R112, R125, R126, R13, R139, R14, R140, R153, R154, R167, R168, R181, R182, R195, R196, R209, R210, R223, R224, R237, R238, R251, R252, R265, R266, R27, R279, R28, R280, R41, R42, R55, R56, R69, R70, R83, R84, R97, R98: value 100k -> 1M

Commit message: Change C6 to DNP
Rise time was slow, causing chip to run bootloader instead of booting from flash
Parts:
- C102, C108, C114, C12, C120, C18, C24, C30, C36, C42, C48, C54, C6, C60, C66, C72, C78, C84, C90, C96: value 0.1uF -> DNP
